File: Hardware/0. Project/Tiny PowerSpy.brd (EAGLE design)
At the start: 42.5 x 32.5 mm, 61 parts, among them U2 SPX3819, U3 ACS712, U4 LMV321, U5 LMV321, U6 NRF52832, Y1 32MHz

Commit message: PCB 1.0 - WIP
Parts:
- added PAD6, PAD7: (no value), Wirepad:SMD2,54-5,08
- added U1: MP100LG, MP100LGN-P:SOIC8E
- C10, C12, C15, C16, C18, C6, C9: device rcl:C0603 -> rcl:C0402
- J2: value (none) -> CORTEX_DEBUGPTH
- PAD1, PAD4: device wirepad:2,15/1,0 -> Wirepad:SMD1,27-2,54
- PAD2, PAD3: device wirepad:2,15/1,0 -> Wirepad:SMD2,54-5,08
- moved R8 143.6 mm to (32.8, 3.71), turned to 90 degrees
- moved R76 142.4 mm to (41.0, 3.71), turned to 270 degrees
- moved Y1 141.7 mm to (11.5, 3.10)
- moved J2 141.2 mm to (40.2, 14.9), turned to 270 degrees
- moved E1 137.8 mm to (6.32, 7.26), turned to 90 degrees
- moved U6 137.5 mm to (18.4, 7.09), turned to 180 degrees
- moved R34 135.6 mm to (32.8, 6.81), turned to 90 degrees
- moved C1 133.3 mm to (34.0, 25.2), flipped to the bottom, turned to 90 degrees
- moved R7 132.4 mm to (24.6, 6.15), flipped to the bottom, turned to 90 degrees
- moved R5 132.4 mm to (27.1, 6.15), flipped to the bottom, turned to 90 degrees
- moved C20 131.4 mm to (17.3, 8.89), flipped to the bottom, turned to 180 degrees
- moved C38 126.6 mm to (36.9, 3.71), turned to 270 degrees
- moved R79 125.7 mm to (38.0, 9.93)
- moved L1 124.6 mm to (39.3, 24.4), flipped to the bottom
- moved C29 121.6 mm to (22.7, 3.48), turned to 270 degrees
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Connections:
- removed net +4.1V: C1.1, C10.1, C11.1, C15.1, C19.1, C20.2, C25.2, C26.1, C38.1, C8.1, J2.1, L1.2, R1.2, R2.2, R76.2, U2.5, U3.8, U4.5, U5.5, U6.13, U6.36, U6.48
- removed net L1_PHASE: F1.1, PAD1.1, R24.1, U3.1, U3.2
- new net 3.3V: C10.1, C11.1, C15.1, C19.1, C25.2, C26.1, C38.1, J2.1, R76.2, U2.5, U4.5, U5.5, U6.13, U6.36, U6.48
- new net IP+: F1.1, PAD3.1, R24.1, U3.1, U3.2
- new net IP-: PAD6.1, U3.3, U3.4
- new net N$16: C5.1, C7.1, L1.1, U2.1, U2.3
- new net PE: PAD4.1, PAD7.1
- net 0V: now also U1.2, U1.9
- net 127V: now also U1.8
- net 5V: now also C1.1, C20.2, C8.1, L1.2, R1.2, R2.2, U1.4, U3.8; no longer C5.1, C7.1, L1.1, U2.1, U2.3
- net ADC_CURRENT: no longer R5.1, U3.7
- net N$1: now also U1.1
- net N$10: now also R5.1, U3.7; no longer PAD3.1, U3.3, U3.4
- net N$4: now also U1.3
- net N$5: now also U1.5, U1.6
- net NEUTRAL: now also PAD1.1; no longer PAD4.1
Routing:
- net 0V: track 0.00 -> 34.0 mm, vias 0 -> 80
- net IP+: track 0.00 -> 22.0 mm, vias 0 -> 1
- net NEUTRAL: track 0.00 -> 20.0 mm
- net 3.3V: track 0.00 -> 12.6 mm
- net N$10: track 0.00 -> 11.7 mm
- net ADC_CURRENT: track 0.00 -> 11.6 mm, vias 0 -> 1
- net N$2: track 0.00 -> 9.64 mm
- net CRYSTAL_XC2: track 0.00 -> 9.42 mm
- net IP-: track 0.00 -> 8.49 mm, vias 0 -> 5
- net N$7: track 0.00 -> 7.88 mm
- net N$3: track 0.00 -> 6.33 mm
- net AGND: track 0.00 -> 5.45 mm
- net N$31: track 0.00 -> 5.32 mm
- net N$9: track 0.00 -> 4.48 mm
- net N$15: track 0.00 -> 4.45 mm
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- added copper zone on layer 16, net IP+
- added copper zone on layer 1, net IP-
- added copper zone on layer 16, net IP-
Other:
- outline, holes or cut-outs redrawn

Commit message: PCB 1.0 - WIP
Parts:
- moved C11 9.49 mm to (40.4, 25.3)
- moved C13 9.49 mm to (35.3, 25.3)
- moved C7 9.49 mm to (37.7, 28.7)
- moved U2 9.49 mm to (37.8, 25.6)
- moved R1 7.67 mm to (30.9, 30.0), turned to 0 degrees
- moved C6 1.55 mm to (22.5, 1.32), turned to 0 degrees
- moved C15 0.82 mm to (26.5, 10.1)
- moved R6 0.51 mm to (13.4, 26.8)
- moved J2 0.49 mm to (39.7, 14.8)
- moved R4 0.43 mm to (9.22, 26.8)
- moved R29 0.43 mm to (23.0, 6.78)
- moved C16 0.18 mm to (13.4, 3.12)
- moved C29 0.11 mm to (22.8, 3.53)
- moved R82 0.10 mm to (39.0, 3.71)
Routing:
- net 3.3V: track 12.6 -> 86.5 mm, vias 0 -> 6
- net NEUTRAL: track 20.0 -> 84.3 mm, vias 0 -> 37
- net 5V: track 1.14 -> 60.1 mm, vias 0 -> 2
- net PE: track 0.00 -> 47.3 mm, vias 0 -> 36
- net 0V: track 34.0 -> 76.6 mm, vias 80 -> 100
- net MCU_SWDIO/TMS: track 0.95 -> 35.6 mm
- net MCU_SWDCLK/TCK: track 1.59 -> 33.8 mm, vias 1 -> 2
- net MCU_SWO/TDO: track 0.00 -> 29.2 mm
- net !MCU_RESET!: track 0.00 -> 25.6 mm
- net ADC_AGND: track 0.00 -> 21.6 mm
- net IP+: track 22.0 -> 41.3 mm, vias 1 -> 2
- net N$5: track 0.00 -> 17.1 mm
- net AGND: track 5.45 -> 16.3 mm
- net N$16: track 0.00 -> 10.6 mm, vias 0 -> 1
- net ADC_CURRENT: track 11.6 -> 18.7 mm
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- added copper zone on layer 1, net 0V
- added copper zone on layer 16, net 0V

Commit message: PCB 1.0 - Done
Parts:
- removed C29: 10nF x 50V, rcl:C0603
- removed C38: 100nF x 50V, rcl:C0603
- removed PAD7: (no value), Wirepad:SMD2,54-5,08
- removed R24: 200k (0.5%), rcl:R0603
- added C21: 6 pF, rcl:C0402
- added C24: DNP, rcl:C0603
- added PAD5: (no value), Wirepad:SMD1,27-2,54
- added R10: 200k (0.5%), rcl:R0603
- C1: value (none) -> 100nF x 50V
- C10: value 100 nF -> (none); device rcl:C0402 -> rcl:E3,5-8
- C11: value 10uF x 10V -> 100nF x 50V
- C12: value DNP -> 100 nF
- C13: value 10nF x 50V -> 100 nF; device rcl:C0603 -> rcl:C0402
- C14: value 1 uF -> 4.7 uF
- C16: value 6 pF -> DNP
- C17: value DNP -> 100 pF; device rcl:C0603 -> rcl:C0402
- C18: value 6 pF -> 1 uF; device rcl:C0402 -> rcl:C0603
- C19: value 4.7 uF -> 10nF x 50V
- C2: device rcl:E3,5-8 -> rcl:C0603
- C20: value 100nF x 50V -> 6 pF; device rcl:C0603 -> rcl:C0402
- C3: value 1nF x 50V -> 100nF x 50V
- C4: value 100nF x 50V -> 100uF x 6.3V; device rcl:C0603 -> rcl:C1206K
- C6: value 100 nF -> 100nF x 50V; device rcl:C0402 -> rcl:C0603
- C7: value 100nF x 50V -> 10nF x 50V
- C8: value 100uF x 6.3V -> 10uF x 10V; device rcl:C1206K -> rcl:C0603
- C9: value 100 pF -> 1nF x 50V; device rcl:C0402 -> rcl:C0603
- PAD1, PAD4: device Wirepad:SMD1,27-2,54 -> Wirepad:SMD2,54-5,08
- PAD3: device Wirepad:SMD2,54-5,08 -> Wirepad:SMD1,27-2,54
- R2: value (none) -> 4k7 (1%)
- R4: value 10R x 1W -> 10k (1%); device resistor pot:0207/5V -> rcl:R0603
- R5: value 4k7 (1%) -> (none)
- R6: value 130V -> 10R x 1W; device varistor:S05K11 -> resistor pot:0207/5V
- R7: value 10k (1%) -> 130V; device rcl:R0603 -> varistor:S05K11
- U1: value MP100LG -> ACS712; device MP100LGN-P:SOIC8E -> ACS712:SOIC127P600X175-8N
- U2: value SPX3819 -> MP100LG; device SPX3819M5-L-3-3:SOT95P280X145-5N -> MP100LGN-P:SOIC8E
- U3: value ACS712 -> SPX3819; device ACS712:SOIC127P600X175-8N -> SPX3819M5-L-3-3:SOT95P280X145-5N
- U4: value LMV321 -> NRF52832; device linear:SOT23-5 -> nrf52832-breakout-temp:QFN48-6X6MM
- U6: value NRF52832 -> LMV321; device nrf52832-breakout-temp:QFN48-6X6MM -> linear:SOT23-5
- moved C6 31.3 mm to (37.7, 28.7)
- moved C11 27.1 mm to (25.7, 2.51), turned to 180 degrees
- moved C4 26.1 mm to (38.2, 27.6)
- moved C10 26.1 mm to (24.3, 28.2), turned to 270 degrees
- moved R4 25.8 mm to (24.6, 6.15), flipped to the bottom, turned to 90 degrees
- moved R7 23.6 mm to (13.4, 26.8), flipped to the top, turned to 180 degrees
- moved C1 23.3 mm to (17.3, 8.89), turned to 180 degrees
- moved R5 23.0 mm to (35.0, 27.8), turned to 0 degrees
- moved U3 21.9 mm to (37.8, 25.6), flipped to the top
- moved R2 21.0 mm to (27.1, 6.15), turned to 90 degrees
- moved U6 19.5 mm to (37.9, 6.93), turned to 90 degrees
- moved PAD1 19.3 mm to (11.8, 16.3)
- moved PAD2 19.3 mm to (11.8, 16.3)
- moved PAD3 19.3 mm to (31.1, 16.3)
- moved C13 17.5 mm to (26.5, 10.1), turned to 0 degrees
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- renumbered C26 to C22, J2 to J1, R25 to R9, R26 to R11, R27 to R12, R29 to R13, R34 to R14, R38 to R15, R39 to R16, R40 to R17, R76 to R18, R79 to R19, R82 to R20
Connections:
- net !MCU_RESET!: now also U4.24; no longer U6.24
- net 0V: now also C1.1, C10.-, C11.1, C20.2, C21.2, C24.2, C25.2, R4.2, R5.1, U1.5, U2.9, U3.2, U4.31, U4.45, U4.EP, U6.2; no longer C10.2, C11.2, C2.-, C20.1, C25.1, C29.2, C38.2, R3.1, R7.2, U1.2, U1.9, U3.5, U4.2, U6.31, U6.45, U6.EP
- net 127V: now also U2.8; no longer U1.8
- net 3.3V: now also C11.2, C12.1, C13.1, C14.1, C25.1, C8.1, U3.5, U4.13, U4.36, U4.48, U6.5; no longer C10.1, C11.1, C15.1, C19.1, C25.2, C38.1, U2.5, U4.5, U6.13, U6.36, U6.48
- net 5V: now also C1.2, C2.1, C4.1, R3.2, U1.8, U2.4; no longer C1.1, C20.2, C8.1, R2.2, U1.4, U3.8
- net ADC_AGND: now also U4.6; no longer U6.6
- net ADC_CURRENT: now also C3.1, R2.2, R4.1, U4.5; no longer C4.1, R5.2, R7.1, U6.5
- net ADC_VOLTAGE: now also C19.1, U4.4; no longer C29.1, U6.4
- net AGND: now also U6.3, U6.4; no longer U5.3, U5.4
- net CRYSTAL_XC1: now also C20.1, U4.34; no longer C16.1, U6.34
- net CRYSTAL_XC2: now also C21.1, U4.35; no longer C18.1, U6.35
- net IP+: now also PAD1.1, R8.1, U1.1, U1.2; no longer PAD3.1, R24.1, U3.1, U3.2
- net IP-: now also PAD2.1, U1.3, U1.4; no longer PAD6.1, U3.3, U3.4
- net MCU_BLE_ANT: now also U4.30; no longer U6.30
- net MCU_SWDCLK/TCK: now also U4.25; no longer U6.25
- net MCU_SWDIO/TMS: now also U4.26; no longer U6.26
- net MCU_SWO/TDO: now also U4.21; no longer U6.21
- net N$1: now also U2.1; no longer U1.1
- net N$10: now also R2.1, U1.7; no longer R5.1, U3.7
- net N$11: now also C24.1; no longer C17.1
- net N$12: now also R10.1; no longer R8.1
- net N$13: now also C17.1, U4.33; no longer C9.1, U6.33
- net N$14: now also R10.2; no longer R8.2
- net N$15: now also U5.4; no longer U4.4
- net N$16: now also C6.1, U3.1, U3.3; no longer C7.1, U2.1, U2.3
- net N$19: now also R8.2; no longer R24.2
- net N$2: now also R7.1; no longer R4.1
- net N$20: now also C7.1, U3.4; no longer C13.1, U2.4
- net N$3: now also C16.1, U4.32; no longer C12.1, U6.32
- net N$30: now also U5.3; no longer U4.3
- net N$32: now also U5.1; no longer U4.1
- net N$4: now also C2.2, R3.1, R5.2, U2.3; no longer C1.2, R2.1, R3.2, U1.3
- net N$5: now also C10.+, U2.5, U2.6; no longer C2.+, U1.5, U1.6
- net N$6: now also C9.1, U1.6; no longer C3.1, U3.6
- net N$7: now also R6.2; no longer R4.2
- net N$76: now also U6.1; no longer U5.1
- net N$8: now also C15.1, U4.1; no longer C6.1, U6.1
- net N$9: now also C18.1, U4.46; no longer C14.1, U6.46
- net NEUTRAL: now also PAD3.1, PAD4.1, R7.2; no longer PAD1.1, PAD2.1, R6.2
- net PE: now also PAD5.1, PAD6.1; no longer PAD4.1, PAD7.1
Routing:
- net ADC_CURRENT: track 18.7 -> 14.7 mm
- net 3.3V: track 86.5 -> 83.3 mm
- net N$15: track 4.80 -> 4.05 mm
