File: Hardware/0. Project/Tiny PowerSpy.sch (EAGLE design)
At the start: 0 parts

Commit message: WIP - Schematic 1.0
Parts:
- added B1: MB6S, rectifier:MB6S
- added C1: (no value), rcl:C-EUC0603
- added C10, C15, C26, C6: 100 nF, rcl:C-EUC0603
- added C11: 10uF x 10V, rcl:C-EUC0603
- added C12, C17: DNP, rcl:C-EUC0603
- added C13, C29: 10nF x 50V, rcl:C-EUC0603
- added C14: 1 uF, rcl:C-EUC0603
- added C16, C18: 6 pF, rcl:C-EUC0603
- added C19: 4.7 uF, rcl:C-EUC0603
- added C2: (no value), rcl:CPOL-EUE3.5-8
- added C20, C25, C38, C4, C7: 100nF x 50V, rcl:C-EUC0603
- added C23: 0.8 pF, rcl:C-EUC0603
- added C3: 1nF x 50V, rcl:C-EUC0603
- added C5, C8: 100uF x 6.3V, rcl:C-USC1206K
- added C9: 100 pF, rcl:C-EUC0603
- added E1: ANT, SparkFun-RF:ANTENNA-GROUNDEDTRACE-15.2MM
- added F1: 250mA, Fuse SMD:0154004.DR
- added J2: CORTEX_DEBUGPTH, SparkFun-Connectors:CORTEX_DEBUGPTH
- added L1: 22uH, rc-master-smd:L_0603
- added L2: 3.9nH, nrf52832-breakout-temp:INDUCTOR-0402-3.9NH
- added PAD1, PAD2, PAD3, PAD4: (no value), wirepad:2,15/1,0
- added R1, R2, R3: (no value), rcl:R-EU_R0603
- added R24, R25, R26, R8: 200k (0.5%), rcl:R-EU_R0603
- added R27: 220R (5%), rcl:R-EU_R0603
- added R29: 47R (5%), rcl:R-EU_R0603
- added R34: 1k4 (0.5%), rcl:R-EU_R0603
- added R38, R79: 0R (1%), rcl:R-EU_R0603
- added R39, R40: 100k (0.5%), rcl:R-EU_R0603
- added R4: 10R x 1W, resistor pot:R-EU_0207/5V
- added R5: 4k7 (1%), rcl:R-EU_R0603
- added R6: 130V, varistor:VARISTOR
- added R7: 10k (1%), rcl:R-EU_R0603
- added R76, R82: 100k (1%), rcl:R-EU_R0603
- added U1: MP100LG, MP100LGN-P:MP100LG
- added U2: SPX3819, SPX3819M5-L-3-3:SPX3819M5-L-3-3
- added U3: ACS712, ACS712:ACS712ELCTR-20A-T
- added U4, U5: LMV321, linear:LMV321M5
- added U6: NRF52832, nrf52832-breakout-temp:NRF52832
- added Y1: 32MHz, nrf52832-breakout-temp:CRYSTAL-32MHZ-SMD-2.0X1.6MM
Connections:
- new net !MCU_RESET!: J2.!RESET, U6.P0.21/RESET
- new net +4.1V: C1.1, C10.1, C11.1, C15.1, C19.1, C20.2, C25.2, C26.1, C38.1, C8.1, J2.VCC, L1.2, R1.2, R2.2, R76.2, U1.VOUT, U2.VOUT, U3.VCC, U4.V+, U5.V+, U6.VDD
- new net 0V: B1.-, C10.2, C11.2, C12.2, C13.2, C14.2, C15.2, C16.2, C17.2, C18.2, C19.2, C2.-, C20.1, C23.2, C25.1, C26.2, C29.2, C3.2, C38.2, C4.2, C5.2, C6.2, C7.2, C8.2, C9.2, E1.GND, J2.GND@3, J2.GND@5, J2.GNDDTCT, R3.1, R7.2, R82.2, U1.GND, U2.GND, U3.GND, U4.V-, U5.V-, U6.VSS
- new net 127V: B1.+, U1.VIN
- new net 5V: C5.1, C7.1, L1.1, U2.EN, U2.VIN
- new net ADC_AGND: R79.2, U6.P0.04/AIN2
- new net ADC_CURRENT: C4.1, R5.1, R5.2, R7.1, U3.VIOUT, U6.P0.03/AIN1
- new net ADC_VOLTAGE: C29.1, R29.1, U6.P0.02/AIN0
- new net AGND: R34.2, R38.2, R39.2, R79.1, U5.-IN, U5.OUT
- new net CRYSTAL_XC1: C16.1, U6.XC1(32MHZ), Y1.2
- new net CRYSTAL_XC2: C18.1, U6.XC2(32MHZ), Y1.1
- new net L1_PHASE: F1.1, PAD1.P, R24.1, U3.IP+
- new net MCU_BLE_ANT: C23.1, L2.2, U6.ANT
- new net MCU_SWDCLK/TCK: J2.SWDCLK/TCK, U6.SWDCLK
- new net MCU_SWDIO/TMS: J2.SWDIO/TMS, U6.SWDIO
- new net MCU_SWO/TDO: J2.SWO/TDO, U6.P0.18
- new net N$1: R1.1, U1.PG
- new net N$10: PAD3.P, U3.IP-
- new net N$11: C17.1, E1.SIGNAL, L2.1
- new net N$12: R25.2, R8.1
- new net N$13: C9.1, U6.DEC3
- new net N$14: R26.1, R8.2
- new net N$15: R29.2, R40.1, U4.OUT
- new net N$19: R24.2, R25.1
- new net N$2: F1.2, R4.1, R6.1
- new net N$20: C13.1, U2.BYP
- new net N$3: C12.1, U6.DEC2
- new net N$30: R39.1, R40.2, U4.-IN
- new net N$31: R26.2, R27.2, R34.1
- new net N$32: R27.1, U4.+IN
- new net N$4: C1.2, R2.1, R3.2, U1.FB
- new net N$5: C2.+, U1.VB, U1.VD
- new net N$6: C3.1, U3.FILTER
- new net N$7: B1.AC1, R4.2
- new net N$76: R76.1, R82.1, U5.+IN
- new net N$8: C6.1, U6.DEC1
- new net N$9: C14.1, U6.DEC4
- new net NEUTRAL: B1.AC2, PAD2.P, PAD4.P, R38.1, R6.2
Other:
- note added: "2.4 GHz Bluetooth Transceiver Interface"
- note added: "AC/DC Full Wave Rectifier"
- note added: "DC/DC Buck Converter"
- note added: "Hall Effect-Based Current Sensor"
- note added: "JTAG/SWD Program and Debug Interface"
- note added: "MCU External Oscillators"
- note added: "Passive Low Pass Filter"
- note added: "Pin 13"
- note added: "Pin 36"
- note added: "Pin 48"
- note added: "Tiny PowerSpy INPUT"
- note added: "Tiny PowerSpy OUTPUT"
- note added: "Virtual Analog Voltage Reference"
- note added: "Voltage Sensor"
- note added: "Vp-max 1,65V"
- note added: "Vref 1,65V"
- note added: "nRF52 SoC (Cortex M4 + Bluetooth 5)"

Commit message: PCB 1.0 - WIP
Parts:
- added PAD6, PAD7: (no value), Wirepad:SMD5
- C10, C12, C15, C16, C18, C6, C9: device rcl:C-EUC0603 -> rcl:C-EUC0402
- PAD1, PAD4: device wirepad:2,15/1,0 -> Wirepad:SMD2
- PAD2, PAD3: device wirepad:2,15/1,0 -> Wirepad:SMD5
Connections:
- removed net +4.1V: C1.1, C10.1, C11.1, C15.1, C19.1, C20.2, C25.2, C26.1, C38.1, C8.1, J2.VCC, L1.2, R1.2, R2.2, R76.2, U1.VOUT, U2.VOUT, U3.VCC, U4.V+, U5.V+, U6.VDD
- removed net L1_PHASE: F1.1, PAD1.P, R24.1, U3.IP+
- new net 3.3V: C10.1, C11.1, C15.1, C19.1, C25.2, C26.1, C38.1, J2.VCC, R76.2, U2.VOUT, U4.V+, U5.V+, U6.VDD
- new net IP+: F1.1, PAD3.P, R24.1, U3.IP+
- new net IP-: PAD6.P, U3.IP-
- new net N$16: C5.1, C7.1, L1.1, U2.EN, U2.VIN
- new net PE: PAD4.P, PAD7.P
- net 5V: now also C1.1, C20.2, C8.1, L1.2, R1.2, R2.2, U1.VOUT, U3.VCC; no longer C5.1, C7.1, L1.1, U2.EN, U2.VIN
- net ADC_CURRENT: no longer R5.1, U3.VIOUT
- net N$10: now also R5.1, U3.VIOUT; no longer PAD3.P, U3.IP-
- net NEUTRAL: now also PAD1.P; no longer PAD4.P
Other:
- moved on the sheet: C25, C29, C38, PAD1, PAD2, PAD3, PAD4, R24, R25, R26, R27, R29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

Commit message: PCB 1.0 - WIP
Changed lines of the file:
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@@
 <part name="R3" library="rcl" library_urn="urn:adsk.eagle:library:334" deviceset="R-EU_" device="R0603" package3d_urn="urn:adsk.eagle:package:23555/3"/>
 <part name="C1" library="rcl" library_urn="urn:adsk.eagle:library:334" deviceset="C-EU" device="C0603" package3d_urn="urn:adsk.eagle:package:23616/2"/>
-<part name="B1" library="rectifier" library_urn="urn:adsk.eagle:library:336" deviceset="MB*S" device="" package3d_urn="urn:adsk.eagle:package:23902/1" technology="6"/>
-<part name="R4" library="resistor pot" deviceset="R-EU_" device="0207/5V" package3d_urn="urn:adsk.eagle:package:20339653/2" value="10R x 1W">
+<part name="B1" library="rectifier" library_urn="urn:adsk.eagle:library:336" deviceset="MB*S" device="" package3d_urn="urn:adsk.eagle:package:23902/1" override_package3d_urn="urn:adsk.eagle:package:22220019/2" override_package_urn="urn:adsk.eagle:footprint:23861/1" technology="6"/>
+<part name="R4" library="resistor pot" deviceset="R-EU_" device="0207/5V" package3d_urn="urn:adsk.eagle:package:20339653/2" override_package3d_urn="urn:adsk.eagle:package:22220755/2" override_package_urn="urn:adsk.eagle:footprint:22995/1" override_locally_modified="yes" value="10R x 1W">
+<spice>
+<pinmapping spiceprefix="R">
+<pinmap gate="G$1" pin="1" pinorder="1"/>
+<pinmap gate="G$1" pin="2" pinorder="2"/>
+</pinmapping>
+</spice>
 <attribute name="PN" value=" AC01000008208JACCS"/>
 </part>
@@
 <part name="C8" library="rcl" deviceset="C-US" device="C1206K" package3d_urn="urn:adsk.eagle:package:23682/2" value="100uF x 6.3V"/>
 <part name="C5" library="rcl" deviceset="C-US" device="C1206K" package3d_urn="urn:adsk.eagle:package:23682/2" value="100uF x 6.3V"/>
-<part name="L1" library="rc-master-smd" deviceset="L_" device="0603" value="22uH"/>
-<part name="U3" library="ACS712" deviceset="ACS712ELCTR-20A-T" device="" value="ACS712"/>
-<part name="F1" library="Fuse SMD" deviceset="0154004.DR" device="" value="250mA"/>
+<part name="L1" library="rc-master-smd" deviceset="L_" device="0603" override_package3d_urn="urn:adsk.eagle:package:22220031/2" override_package_urn="urn:adsk.eagle:footprint:22220032/1" value="22uH"/>
+<part name="U3" library="ACS712" deviceset="ACS712ELCTR-20A-T" device="" override_package3d_urn="urn:adsk.eagle:package:22219930/2" override_package_urn="urn:adsk.eagle:footprint:22219931/1" value="ACS712"/>
+<part name="F1" library="Fuse SMD" deviceset="0154004.DR" device="" override_package3d_urn="urn:adsk.eagle:package:22220010/2" override_package_urn="urn:adsk.eagle:footprint:22220011/1" value="250mA"/>
 <part name="C2" library="rcl" deviceset="CPOL-EU" device="E3.5-8" package3d_urn="urn:adsk.eagle:package:23360/2"/>
 <part name="U4" library="linear" deviceset="LMV321?*" device="M5" package3d_urn="urn:adsk.eagle:package:16456/2" value="LMV321"/>
@@
 <part name="SUPPLY4" library="supply2" library_urn="urn:adsk.eagle:library:372" deviceset="+4.1V" device="" value="3.3V"/>
 <part name="SUPPLY5" library="supply2" library_urn="urn:adsk.eagle:library:372" deviceset="+4.1V" device="" value="3.3V"/>
-<part name="L2" library="nrf52832-breakout-temp" deviceset="INDUCTOR" device="-0402-3.9NH" value="3.9nH"/>
-<part name="J2" library="SparkFun-Connectors" deviceset="CORTEX_DEBUG" device="PTH" value="CORTEX_DEBUGPTH"/>
+<part name="L2" library="nrf52832-breakout-temp" deviceset="INDUCTOR" device="-0402-3.9NH" override_package3d_urn="urn:adsk.eagle:package:22220041/2" override_package_urn="urn:adsk.eagle:footprint:22220042/1" value="3.9nH"/>
+<part name="J2" library="SparkFun-Connectors" deviceset="CORTEX_DEBUG" device="PTH" override_package3d_urn="urn:adsk.eagle:package:22220046/2" override_package_urn="urn:adsk.eagle:footprint:22220047/1" value="CORTEX_DEBUGPTH"/>
 <part name="GND11" library="supply1" library_urn="urn:adsk.eagle:library:371" deviceset="0V" device=""/>
 <part name="GND12" library="supply1" library_urn="urn:adsk.eagle:library:371" deviceset="0V" device=""/>
@@
 <attribute name="PN" value="RC0603DR-07200KL"/>
 </part>
-<part name="U6" library="nrf52832-breakout-temp" deviceset="NRF52832" device=""/>
+<part name="U6" library="nrf52832-breakout-temp" deviceset="NRF52832" device="" override_package3d_urn="urn:adsk.eagle:package:22219961/2" override_package_urn="urn:adsk.eagle:footprint:22219962/1"/>
 <part name="E1" library="SparkFun-RF" deviceset="ANTENNA-GROUNDED" device="TRACE-15.2MM" value="ANT"/>
-<part name="Y1" library="nrf52832-breakout-temp" deviceset="CRYSTAL-32MHZ" device="-SMD-2.0X1.6MM" value="32MHz"/>
+<part name="Y1" library="nrf52832-breakout-temp" deviceset="CRYSTAL-32MHZ" device="-SMD-2.0X1.6MM" override_package3d_urn="urn:adsk.eagle:package:22219997/2" override_package_urn="urn:adsk.eagle:footprint:22219998/1" value="32MHz"/>
 <part name="PAD1" library="Wirepad" deviceset="SMD2" device="" package3d_urn="urn:adsk.eagle:package:30839/1"/>
 <part name="PAD4" library="Wirepad" deviceset="SMD2" device="" package3d_urn="urn:adsk.eagle:package:30839/1"/>
@@
 <part name="PAD6" library="Wirepad" deviceset="SMD5" device="" package3d_urn="urn:adsk.eagle:package:30841/1"/>
 <part name="PAD3" library="Wirepad" deviceset="SMD5" device="" package3d_urn="urn:adsk.eagle:package:30841/1"/>
-<part name="U1" library="MP100LGN-P" deviceset="MP100LG" device=""/>
+<part name="U1" library="MP100LGN-P" deviceset="MP100LG" device="" override_package3d_urn="urn:adsk.eagle:package:22219955/2" override_package_urn="urn:adsk.eagle:footprint:22219956/1"/>
 </parts>
 <sheets>
@@
 </instance>
 <instance part="E1" gate="G$1" x="375.92" y="69.85" smashed="yes">
-<attribute name="NAME" x="384.81" y="68.072" size="1.778" layer="95" font="vector" rot="MR0"/>
-<attribute name="VALUE" x="384.81" y="65.786" size="1.778" layer="96" font="vector" rot="MR0"/>
+<attribute name="NAME" x="374.015" y="72.263" size="1.778" layer="95" font="vector" rot="MR180"/>
+<attribute name="VALUE" x="374.015" y="74.549" size="1.778" layer="96" font="vector" rot="MR180"/>
 </instance>
 <instance part="Y1" gate="G$1" x="210.185" y="62.865" smashed="yes" rot="MR0">
@@
 packages will not be understood (or retained) with this version.
 </note>
+<note version="9.4" severity="warning">
+Since Version 9.4, EAGLE supports the overriding of 3D packages
+in schematics and board files. Those overridden 3d packages
+will not be understood (or retained) with this version.
+</note>
 <note version="8.4" severity="warning">

Commit message: PCB 1.0 - Done
Parts:
- removed C29: 10nF x 50V, rcl:C-EUC0603
- removed C38: 100nF x 50V, rcl:C-EUC0603
- removed PAD7: (no value), Wirepad:SMD5
- removed R24: 200k (0.5%), rcl:R-EU_R0603
- added C21: 6 pF, rcl:C-EUC0402
- added C24: DNP, rcl:C-EUC0603
- added PAD5: (no value), Wirepad:SMD2
- added R10: 200k (0.5%), rcl:R-EU_R0603
- C1: value (none) -> 100nF x 50V; PN (none) -> C0603C104M5RACTU
- C10: value 100 nF -> (none); device rcl:C-EUC0402 -> rcl:CPOL-EUE3.5-8
- C11: value 10uF x 10V -> 100nF x 50V; PN GRM188R61A106ME69D -> C0603C104M5RACTU
- C12: value DNP -> 100 nF
- C13: value 10nF x 50V -> 100 nF; device rcl:C-EUC0603 -> rcl:C-EUC0402; PN C0603C103M5RACTU -> (none)
- C14: value 1 uF -> 4.7 uF
- C16: value 6 pF -> DNP
- C17: value DNP -> 100 pF; device rcl:C-EUC0603 -> rcl:C-EUC0402
- C18: value 6 pF -> 1 uF; device rcl:C-EUC0402 -> rcl:C-EUC0603
- C19: value 4.7 uF -> 10nF x 50V; PN (none) -> C0603C103M5RACTU
- C2: device rcl:CPOL-EUE3.5-8 -> rcl:C-EUC0603
- C20: value 100nF x 50V -> 6 pF; device rcl:C-EUC0603 -> rcl:C-EUC0402; PN C0603C104M5RACTU -> (none)
- C3: value 1nF x 50V -> 100nF x 50V
- C4: value 100nF x 50V -> 100uF x 6.3V; device rcl:C-EUC0603 -> rcl:C-USC1206K; PN C0603C104M5RACTU -> (none)
- C6: value 100 nF -> 100nF x 50V; device rcl:C-EUC0402 -> rcl:C-EUC0603; PN (none) -> C0603C104M5RACTU
- C7: value 100nF x 50V -> 10nF x 50V; PN C0603C104M5RACTU -> C0603C103M5RACTU
- C8: value 100uF x 6.3V -> 10uF x 10V; device rcl:C-USC1206K -> rcl:C-EUC0603; PN (none) -> GRM188R61A106ME69D
- C9: value 100 pF -> 1nF x 50V; device rcl:C-EUC0402 -> rcl:C-EUC0603; PN (none) -> C0603C104M5RACTU
- PAD1, PAD4: device Wirepad:SMD2 -> Wirepad:SMD5
- PAD3: device Wirepad:SMD5 -> Wirepad:SMD2
- R2: value (none) -> 4k7 (1%)
- R4: value 10R x 1W -> 10k (1%); device resistor pot:R-EU_0207/5V -> rcl:R-EU_R0603; PN AC01000008208JACCS -> (none)
- R5: value 4k7 (1%) -> (none)
- R6: value 130V -> 10R x 1W; device varistor:VARISTOR -> resistor pot:R-EU_0207/5V; PN (none) -> AC01000008208JACCS
- R7: value 10k (1%) -> 130V; device rcl:R-EU_R0603 -> varistor:VARISTOR
- U1: value MP100LG -> ACS712; device MP100LGN-P:MP100LG -> ACS712:ACS712ELCTR-20A-T
- U2: value SPX3819 -> MP100LG; device SPX3819M5-L-3-3:SPX3819M5-L-3-3 -> MP100LGN-P:MP100LG; PN SPX3819M5-L-3-3/TR -> (none)
- U3: value ACS712 -> SPX3819; device ACS712:ACS712ELCTR-20A-T -> SPX3819M5-L-3-3:SPX3819M5-L-3-3; PN (none) -> SPX3819M5-L-3-3/TR
- U4: value LMV321 -> NRF52832; device linear:LMV321M5 -> nrf52832-breakout-temp:NRF52832
- U6: value NRF52832 -> LMV321; device nrf52832-breakout-temp:NRF52832 -> linear:LMV321M5
- renumbered C26 to C22, J2 to J1, R25 to R9, R26 to R11, R27 to R12, R29 to R13, R34 to R14, R38 to R15, R39 to R16, R40 to R17, R76 to R18, R79 to R19, R82 to R20
Connections:
- net !MCU_RESET!: now also U4.P0.21/RESET; no longer U6.P0.21/RESET
- net 0V: now also C1.1, C10.-, C11.1, C20.2, C21.2, C24.2, C25.2, R4.2, R5.1, U4.VSS, U6.V-; no longer C10.2, C11.2, C2.-, C20.1, C25.1, C29.2, C38.2, R3.1, R7.2, U4.V-, U6.VSS
- net 127V: now also U2.VIN; no longer U1.VIN
- net 3.3V: now also C11.2, C12.1, C13.1, C14.1, C25.1, C8.1, U3.VOUT, U4.VDD, U6.V+; no longer C10.1, C11.1, C15.1, C19.1, C25.2, C38.1, U2.VOUT, U4.V+, U6.VDD
- net 5V: now also C1.2, C2.1, C4.1, R3.2, U1.VCC, U2.VOUT; no longer C1.1, C20.2, C8.1, R2.2, U1.VOUT, U3.VCC
- net ADC_AGND: now also U4.P0.04/AIN2; no longer U6.P0.04/AIN2
- net ADC_CURRENT: now also C3.1, R2.2, R4.1, U4.P0.03/AIN1; no longer C4.1, R5.2, R7.1, U6.P0.03/AIN1
- net ADC_VOLTAGE: now also C19.1, U4.P0.02/AIN0; no longer C29.1, U6.P0.02/AIN0
- net AGND: now also U6.-IN, U6.OUT; no longer U5.-IN, U5.OUT
- net CRYSTAL_XC1: now also C20.1, U4.XC1(32MHZ); no longer C16.1, U6.XC1(32MHZ)
- net CRYSTAL_XC2: now also C21.1, U4.XC2(32MHZ); no longer C18.1, U6.XC2(32MHZ)
- net IP+: now also PAD1.P, R8.1, U1.IP+; no longer PAD3.P, R24.1, U3.IP+
- net IP-: now also PAD2.P, U1.IP-; no longer PAD6.P, U3.IP-
- net MCU_BLE_ANT: now also U4.ANT; no longer U6.ANT
- net MCU_SWDCLK/TCK: now also U4.SWDCLK; no longer U6.SWDCLK
- net MCU_SWDIO/TMS: now also U4.SWDIO; no longer U6.SWDIO
- net MCU_SWO/TDO: now also U4.P0.18; no longer U6.P0.18
- net N$1: now also U2.PG; no longer U1.PG
- net N$10: now also R2.1, U1.VIOUT; no longer R5.1, U3.VIOUT
- net N$11: now also C24.1; no longer C17.1
- net N$12: now also R10.1; no longer R8.1
- net N$13: now also C17.1, U4.DEC3; no longer C9.1, U6.DEC3
- net N$14: now also R10.2; no longer R8.2
- net N$15: now also U5.OUT; no longer U4.OUT
- net N$16: now also C6.1, U3.EN, U3.VIN; no longer C7.1, U2.EN, U2.VIN
- net N$19: now also R8.2; no longer R24.2
- net N$2: now also R7.1; no longer R4.1
- net N$20: now also C7.1, U3.BYP; no longer C13.1, U2.BYP
- net N$3: now also C16.1, U4.DEC2; no longer C12.1, U6.DEC2
- net N$30: now also U5.-IN; no longer U4.-IN
- net N$32: now also U5.+IN; no longer U4.+IN
- net N$4: now also C2.2, R3.1, R5.2, U2.FB; no longer C1.2, R2.1, R3.2, U1.FB
- net N$5: now also C10.+, U2.VB, U2.VD; no longer C2.+, U1.VB, U1.VD
- net N$6: now also C9.1, U1.FILTER; no longer C3.1, U3.FILTER
- net N$7: now also R6.2; no longer R4.2
- net N$76: now also U6.+IN; no longer U5.+IN
- net N$8: now also C15.1, U4.DEC1; no longer C6.1, U6.DEC1
- net N$9: now also C18.1, U4.DEC4; no longer C14.1, U6.DEC4
- net NEUTRAL: now also PAD3.P, PAD4.P, R7.2; no longer PAD1.P, PAD2.P, R6.2
- net PE: now also PAD5.P, PAD6.P; no longer PAD4.P, PAD7.P
Other:
- moved on the sheet: C1, C11, C12, C13, C14, C15, C16, C17, C18, C19, C20, C25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
